Commit message: feat(ippolit_description): A4 -- URDF as single source of robot geometry
Measured the robot's real geometry (tape measure) and encoded it in one
xacro <property> block: chassis radius 0.175m, LDS turret 0.095m high at
center, camera 0.16m fwd / 0.06m high / centered, camera yaw 1.8deg (from
F0(b)/G26). The URDF is now the one source of geometry truth.

Removed duplicated static-TF publishers:
- q6a_laser_odom no longer publishes its own base_link->laser identity TF
  (the URDF owns it now, with the real height). robot_state_publisher is
  the sole /tf_static publisher. Dropped the orphaned laser_frame param.
- q6a_objmap drops its cam_yaw_deg param and reads the camera yaw from the
  URDF via a base_link->camera_link TF lookup (cached, 0-yaw fallback).
  cam_hfov_deg stays a param (sensor intrinsic). Added yaw_from_quaternion
  + 4 unit tests.

Verified live: view_frames shows the tree sourced from URDF, tf2_echo
confirms the measured offsets, objmap logs "camera yaw from TF: 1.80 deg".
20/20 colcon test green. Wheel base deliberately not encoded (no consumer
yet -- we drive via Valetudo REST, /odom_laser is scan-matched).

Co-Authored-By: Claude Sonnet 5 <noreply@anthropic.com>

File: ros2_ws/src/ippolit_description/urdf/ippolit.urdf.xacro (robot description, xacro)
@@ -1,13 +1,34 @@
 <?xml version="1.0"?>
 <!--
-  ippolit.urdf.xacro — placeholder robot description, scaffolded in A0.
-  Geometry below uses only values already known from live calibration (docs/navigation-architecture.md
-  §8 appendix): chassis diameter ~0.350m (spec) / BODY_R=0.219m (empirical clearance offset, NOT the same
-  thing — see q6a_creep_test.py's history comment for why they differ and are still unreconciled).
-  laser/camera poses are UNMEASURED placeholders (0,0,0) pending F0.2 (camera bearing/FOV calibration)
-  and the A4 step that's supposed to replace every ad-hoc static-TF publish in the codebase with this
-  file as the single source of geometry truth. Do not trust laser/camera offsets below for anything yet.
+  ippolit.urdf.xacro — the single source of truth for the robot's physical geometry (A4).
+  Every measured constant lives in the xacro <property> block below and NOWHERE else in the
+  codebase: nodes that need a frame relationship look it up via TF (published by
+  robot_state_publisher from this file), rather than hard-coding an offset. This replaced the
+  ad-hoc static base_link->laser TF that q6a_laser_odom used to publish itself (A4 removed it — two
+  publishers of the same static transform with different values is a real bug, cf. the /map
+  double-publisher, G25).
+  Frame convention (REP-103): base_link at the round chassis's geometric center, projected to the
+  FLOOR (z=0 = floor), x forward (direction of travel), y left, z up.
+  Measured live 2026-07-13 (A4), with a tape measure unless noted:
+    - chassis diameter 0.350 m (Dreame D10s Pro spec, confirmed) -> radius 0.175 m
+    - LDS turret scan-slot height 0.095 m above floor; turret sits at the chassis center (x=y=0)
+    - OV8856 camera: 0.16 m forward of center, 0.06 m above floor, on the centerline (y=0)
+    - camera yaw offset 1.8 deg, from F0(b)'s bearing/FOV calibration (G26) — the camera is very
+      slightly rotated vs base_link forward; this is the SAME 1.8 deg objmap used to apply as its
+      cam_yaw_deg param, now sourced here instead (objmap reads it back from TF — A4).
+  Camera HFOV (116.7 deg, G26) is a sensor INTRINSIC, not a frame pose, so it stays a q6a_objmap
+  parameter — it does not belong in the TF tree.
 -->
 <robot name="ippolit" xmlns:xacro="http://www.ros.org/wiki/xacro">
+  <!-- ===== measured geometry (single source of truth) ===== -->
+  <xacro:property name="chassis_radius" value="0.175"/>
+  <xacro:property name="chassis_height" value="0.097"/>
+  <xacro:property name="laser_x" value="0.0"/>
+  <xacro:property name="laser_y" value="0.0"/>
+  <xacro:property name="laser_z" value="0.095"/>
+  <xacro:property name="camera_x" value="0.16"/>
+  <xacro:property name="camera_y" value="0.0"/>
+  <xacro:property name="camera_z" value="0.06"/>
+  <xacro:property name="camera_yaw" value="${radians(1.8)}"/>
   <material name="chassis_grey">
     <color rgba="0.6 0.6 0.6 1.0"/>
@@ -15,35 +36,39 @@
   <link name="base_link">
     <visual>
-      <origin xyz="0 0 0.04" rpy="0 0 0"/>
+      <origin xyz="0 0 ${chassis_height/2}" rpy="0 0 0"/>
       <geometry>
-        <cylinder radius="0.175" length="0.08"/>
+        <cylinder radius="${chassis_radius}" length="${chassis_height}"/>
       </geometry>
       <material name="chassis_grey"/>
     </visual>
     <collision>
-      <origin xyz="0 0 0.04" rpy="0 0 0"/>
+      <origin xyz="0 0 ${chassis_height/2}" rpy="0 0 0"/>
       <geometry>
-        <cylinder radius="0.175" length="0.08"/>
+        <cylinder radius="${chassis_radius}" length="${chassis_height}"/>
       </geometry>
     </collision>
     <inertial>
       <mass value="3.0"/>
-      <origin xyz="0 0 0.04"/>
+      <origin xyz="0 0 ${chassis_height/2}"/>
       <inertia ixx="0.02" ixy="0" ixz="0" iyy="0.02" iyz="0" izz="0.03"/>
     </inertial>
   </link>
-  <!-- LDS turret: TODO A4 — measure real x/y/z offset from base_link center; 0.0 height placeholder -->
+  <!-- LDS turret. Rotation is identity: lds_scan_node already rotates raw LDS bearings into the
+       base_link convention (ANGLE_OFFSET_DEG), so /scan in frame 'laser' is rotationally aligned
+       to base_link — only the height offset is real. -->
   <link name="laser"/>
   <joint name="laser_joint" type="fixed">
     <parent link="base_link"/>
     <child link="laser"/>
-    <origin xyz="0 0 0.09" rpy="0 0 0"/>
+    <origin xyz="${laser_x} ${laser_y} ${laser_z}" rpy="0 0 0"/>
   </joint>
-  <!-- OV8856 camera: TODO A4/F0.2 — HFOV/yaw calibration feeds this pose; currently a guess -->
+  <!-- OV8856 forward camera. camera_link x-axis = the optical/forward axis; the small yaw is the
+       F0(b)-calibrated misalignment vs base_link forward. q6a_objmap reads this frame's yaw from
+       TF for its bearing math (A4). -->
   <link name="camera_link"/>
   <joint name="camera_joint" type="fixed">
     <parent link="base_link"/>
     <child link="camera_link"/>
-    <origin xyz="0.15 0 0.05" rpy="0 0 0"/>
+    <origin xyz="${camera_x} ${camera_y} ${camera_z}" rpy="0 0 ${camera_yaw}"/>
   </joint>
 </robot>

Commit message: feat(ippolit_localization): EKF wheel+IMU odometry (robot_localization)
Fuse /odom/wheel (AVA MCU wheel odom, was decoded+live but unused) +
/imu/data (gyro) into a smooth odom->base_link via robot_localization,
replacing q6a_laser_odom's scan-matching as the odom source. Key win:
wheel+IMU works without the LiDAR, so odom stays valid during
manual_control when the fanoff gate parks the turret.

- Added imu_link to the URDF (EKF needs the frame; identity offset ok
  for 2D yaw-rate fusion).
- mcu_node now populates covariances on /odom/wheel + /imu/data (RL
  can't fuse zero-covariance messages).
- New ekf.yaml + ekf_node in localization.launch.xml.
- q6a_laser_odom gains publish_tf param (set false): keeps publishing
  /odom_laser as a scan-matched reference but yields odom->base_link to
  the EKF (avoids the two-parents bug, G27).

Verified live: sole odom->base_link publisher, EKF translation matches
raw wheel odom (0.219 vs 0.218m). G28: differential mode over-reported
2x -- fixed with differential:false. G29: exposed that the robot drives
erratically under manual control (inconsistent distance, spontaneous
~75deg turns on a straight command) -- an ACTUATION problem, not
odometry (the EKF tracked each actual path faithfully). F3/F4 will need
closed-loop heading control or that root-caused.

Co-Authored-By: Claude Sonnet 5 <noreply@anthropic.com>

File: ros2_ws/src/ippolit_description/urdf/ippolit.urdf.xacro (robot description, xacro)
@@ -72,3 +72,14 @@
     <origin xyz="${camera_x} ${camera_y} ${camera_z}" rpy="0 0 ${camera_yaw}"/>
   </joint>
+  <!-- BMI055 IMU (on the MCU board). The EKF (robot_localization, wheel+IMU fusion) needs this
+       frame in TF. Exact mount offset is unmeasured, but for the 2D yaw-rate fusion we actually
+       use it doesn't matter: angular velocity is identical everywhere on a rigid body, so an
+       identity offset is correct for our purposes. Axes are assumed base_link-aligned (mcu_node
+       already treats the gyro z as yaw rate); revisit if RViz shows a rotation mismatch. -->
+  <link name="imu_link"/>
+  <joint name="imu_joint" type="fixed">
+    <parent link="base_link"/>
+    <child link="imu_link"/>
+    <origin xyz="0 0 0" rpy="0 0 0"/>
+  </joint>
 </robot>
